Commit message: Trying to adapt limits.

File: nico_upper_rh6d_r.urdf (robot description, URDF)
Before this commit: robot nico_upper_rh6d, 20 links, 19 joints
Joints:
- joint gripper_rjoint: limit lower=-2.57 upper=0 effort=30 velocity=1 -> (none)
- joint r_wrist_x_rjoint: limit lower=-.78 upper=0.78 effort=30 velocity=1 -> lower=-0.785398 upper=0 effort=30 velocity=1
- joint r_wrist_z_rjoint: limit lower=-1.571 upper=1.571 effort=30 velocity=1 -> lower=2.44346 upper=2.6529 effort=30 velocity=1

Commit message: Correcting shoulder limit so it doesn't go below 0.

File: nico_upper_rh6d_r.urdf (robot description, URDF)
Before this commit: robot nico_upper_rh6d, 20 links, 19 joints
Joints:
- joint r_shoulder_y_rjoint: limit lower=-0.5236 upper=3.1416 effort=30 velocity=1 -> lower=0 upper=3.1416 effort=30 velocity=1

Commit message: Fixing limits for wrist_z.

File: nico_upper_rh6d_r.urdf (robot description, URDF)
Before this commit: robot nico_upper_rh6d, 20 links, 19 joints
Joints:
- joint r_wrist_z_rjoint: limit lower=2.44346 upper=2.6529 effort=30 velocity=1 -> lower=1.46608 upper=1.67552 effort=30 velocity=1

Commit message: Entering correct limits and recalculating.

File: nico_upper_rh6d_r.urdf (robot description, URDF)
Before this commit: robot nico_upper_rh6d, 20 links, 19 joints
Joints:
- joint r_wrist_x_rjoint: limit lower=-0.785398 upper=0 effort=30 velocity=1 -> lower=-0.872665 upper=-0.523599 effort=30 velocity=1
- joint r_wrist_z_rjoint: limit lower=1.46608 upper=1.67552 effort=30 velocity=1 -> lower=1.22173 upper=1.5708 effort=30 velocity=1
